Commit message: fix(urdf): Correct mechanical, effort and velicity limits
- Adjust the direction of some joint to make it consistent with raw angle

File: left_hands/d5_left_hands_tips.urdf (robot description, URDF)
Before this commit: robot D5_left_hands_tips, 26 links, 25 joints
Joints:
- joint F1J1: axis 0 0.090031 -0.99594 -> 0 -0.090031 0.99594; limit lower=-1.83 upper=0.52 effort=10000 velocity=10000 -> lower=-0.0448 upper=1.6508 effort=0.6 velocity=8.58701992
- joint F1J2: limit lower=-0.52 upper=1.83 effort=10000 velocity=10000 -> lower=-0.1659 upper=0.9339 effort=0.6 velocity=11.10029404
- joint F1J3: limit lower=-0.52 upper=1.83 effort=10000 velocity=10000 -> lower=-0.4932 upper=1.6272 effort=0.3 velocity=12.86307659
- joint F1J4: limit lower=-0.52 upper=1.83 effort=10000 velocity=10000 -> lower=-0.4932 upper=1.6272 effort=0.3 velocity=13.57866158
- joint F2J1: limit lower=-1.83 upper=0.52 effort=10000 velocity=10000 -> lower=-1.63595 upper=0.32695 effort=1.0 velocity=8.203047484
- joint F2J2: limit lower=-0.52 upper=0.52 effort=10000 velocity=10000 -> lower=-0.495 upper=0.495 effort=0.2 velocity=8.115781022
- joint F2J3: limit lower=-0.52 upper=1.83 effort=10000 velocity=10000 -> lower=-0.4932 upper=1.6272 effort=0.3 velocity=12.86307659
- joint F2J4: limit lower=-0.52 upper=1.83 effort=10000 velocity=10000 -> lower=-0.4932 upper=1.6272 effort=0.3 velocity=13.57866158
- joint F3J1: limit lower=-1.83 upper=0.52 effort=10000 velocity=10000 -> lower=-1.63595 upper=0.32695 effort=1.0 velocity=8.203047484
- joint F3J2: limit lower=-0.52 upper=0.52 effort=10000 velocity=10000 -> lower=-0.495 upper=0.495 effort=0.2 velocity=8.115781022
- joint F3J3: limit lower=-0.52 upper=1.83 effort=10000 velocity=10000 -> lower=-0.4932 upper=1.6272 effort=0.3 velocity=12.86307659
- joint F3J4: limit lower=-0.52 upper=1.83 effort=10000 velocity=10000 -> lower=-0.4932 upper=1.6272 effort=0.3 velocity=13.57866158
- joint F4J1: limit lower=-1.83 upper=0.52 effort=10000 velocity=10000 -> lower=-1.63595 upper=0.32695 effort=1.0 velocity=8.203047484
- joint F4J2: limit lower=-0.52 upper=0.52 effort=10000 velocity=10000 -> lower=-0.495 upper=0.495 effort=0.2 velocity=8.115781022
- joint F4J3: limit lower=-0.52 upper=1.83 effort=10000 velocity=10000 -> lower=-0.4932 upper=1.6272 effort=0.3 velocity=12.86307659
- joint F4J4: limit lower=-0.52 upper=1.83 effort=10000 velocity=10000 -> lower=-0.4932 upper=1.6272 effort=0.3 velocity=13.57866158
- joint F5J1: limit lower=-1.83 upper=0.52 effort=10000 velocity=10000 -> lower=-1.63595 upper=0.32695 effort=1.0 velocity=8.203047484
- joint F5J2: limit lower=-0.52 upper=0.52 effort=10000 velocity=10000 -> lower=-0.495 upper=0.495 effort=0.2 velocity=8.115781022
- joint F5J3: limit lower=-0.5222 upper=1.83 effort=10000 velocity=10000 -> lower=-0.4932 upper=1.6272 effort=0.3 velocity=12.86307659
- joint F5J4: limit lower=-0.52 upper=1.83 effort=10000 velocity=10000 -> lower=-0.4932 upper=1.6272 effort=0.3 velocity=13.57866158

File: left_hands/urdf/d5_left_hands_tips.urdf (robot description, URDF)
Before this commit: robot d5_left_hands_tips, 26 links, 25 joints
Joints:
- joint F1J1: axis 0 0.090031 -0.99594 -> 0 -0.090031 0.99594; limit lower=-1.83 upper=0.52 effort=10000 velocity=10000 -> lower=-0.0448 upper=1.6508 effort=0.6 velocity=8.58701992
- joint F1J2: limit lower=-0.52 upper=1.83 effort=10000 velocity=10000 -> lower=-0.1659 upper=0.9339 effort=0.6 velocity=11.10029404
- joint F1J3: limit lower=-0.52 upper=1.83 effort=10000 velocity=10000 -> lower=-0.4932 upper=1.6272 effort=0.3 velocity=12.86307659
- joint F1J4: limit lower=-0.52 upper=1.83 effort=10000 velocity=10000 -> lower=-0.4932 upper=1.6272 effort=0.3 velocity=13.57866158
- joint F2J1: limit lower=-1.83 upper=0.52 effort=10000 velocity=10000 -> lower=-1.63595 upper=0.32695 effort=1.0 velocity=8.203047484
- joint F2J2: limit lower=-0.52 upper=0.52 effort=10000 velocity=10000 -> lower=-0.495 upper=0.495 effort=0.2 velocity=8.115781022
- joint F2J3: limit lower=-0.52 upper=1.83 effort=10000 velocity=10000 -> lower=-0.4932 upper=1.6272 effort=0.3 velocity=12.86307659
- joint F2J4: limit lower=-0.52 upper=1.83 effort=10000 velocity=10000 -> lower=-0.4932 upper=1.6272 effort=0.3 velocity=13.57866158
- joint F3J1: limit lower=-1.83 upper=0.52 effort=10000 velocity=10000 -> lower=-1.63595 upper=0.32695 effort=1.0 velocity=8.203047484
- joint F3J2: limit lower=-0.52 upper=0.52 effort=10000 velocity=10000 -> lower=-0.495 upper=0.495 effort=0.2 velocity=8.115781022
- joint F3J3: limit lower=-0.52 upper=1.83 effort=10000 velocity=10000 -> lower=-0.4932 upper=1.6272 effort=0.3 velocity=12.86307659
- joint F3J4: limit lower=-0.52 upper=1.83 effort=10000 velocity=10000 -> lower=-0.4932 upper=1.6272 effort=0.3 velocity=13.57866158
- joint F4J1: limit lower=-1.83 upper=0.52 effort=10000 velocity=10000 -> lower=-1.63595 upper=0.32695 effort=1.0 velocity=8.203047484
- joint F4J2: limit lower=-0.52 upper=0.52 effort=10000 velocity=10000 -> lower=-0.495 upper=0.495 effort=0.2 velocity=8.115781022
- joint F4J3: limit lower=-0.52 upper=1.83 effort=10000 velocity=10000 -> lower=-0.4932 upper=1.6272 effort=0.3 velocity=12.86307659
- joint F4J4: limit lower=-0.52 upper=1.83 effort=10000 velocity=10000 -> lower=-0.4932 upper=1.6272 effort=0.3 velocity=13.57866158
- joint F5J1: limit lower=-1.83 upper=0.52 effort=10000 velocity=10000 -> lower=-1.63595 upper=0.32695 effort=1.0 velocity=8.203047484
- joint F5J2: limit lower=-0.52 upper=0.52 effort=10000 velocity=10000 -> lower=-0.495 upper=0.495 effort=0.2 velocity=8.115781022
- joint F5J3: limit lower=-0.5222 upper=1.83 effort=10000 velocity=10000 -> lower=-0.4932 upper=1.6272 effort=0.3 velocity=12.86307659
- joint F5J4: limit lower=-0.52 upper=1.83 effort=10000 velocity=10000 -> lower=-0.4932 upper=1.6272 effort=0.3 velocity=13.57866158

File: right_hands/d5_right_hands_tips.urdf (robot description, URDF)
Before this commit: robot d5_right_hands_tips, 26 links, 25 joints
Joints:
- joint F1J1: axis 0 0 -1 -> 0 0 1; limit lower=-1.83 upper=1 effort=1000 velocity=1000 -> lower=-0.0448 upper=1.6508 effort=0.6 velocity=8.58701992
- joint F1J2: axis 0 1 0 -> 0 -1 0; limit lower=-0.47 upper=1.73 effort=1000 velocity=1000 -> lower=-0.1659 upper=0.9339 effort=0.6 velocity=11.10029404
- joint F1J3: axis 0 0 -1 -> 0 0 1; limit lower=-1.83 upper=0.52 effort=1000 velocity=1000 -> lower=-0.4932 upper=1.6272 effort=0.3 velocity=12.86307659
- joint F1J4: axis 0 0 -1 -> 0 0 1; limit lower=-1.74 upper=0.61 effort=1000 velocity=1000 -> lower=-0.4932 upper=1.6272 effort=0.3 velocity=13.57866158
- joint F2J1: axis 0 0 1 -> 0 0 -1; limit lower=-0.52 upper=1.83 effort=1000 velocity=1000 -> lower=-1.63595 upper=0.32695 effort=1.0 velocity=8.203047484
- joint F2J2: axis 0 -1 0 -> 0 1 0; limit lower=-0.52 upper=0.52 effort=1000 velocity=1000 -> lower=-0.495 upper=0.495 effort=0.2 velocity=8.115781022
- joint F2J3: limit lower=-0.52 upper=1.83 effort=1000 velocity=1000 -> lower=-0.4932 upper=1.6272 effort=0.3 velocity=12.86307659
- joint F2J4: limit lower=-0.52 upper=1.74 effort=1000 velocity=1000 -> lower=-0.4932 upper=1.6272 effort=0.3 velocity=13.57866158
- joint F3J1: axis 0 0 1 -> 0 0 -1; limit lower=-0.52 upper=1.83 effort=1000 velocity=1000 -> lower=-1.63595 upper=0.32695 effort=1.0 velocity=8.203047484
- joint F3J2: axis 0 -1 0 -> 0 1 0; limit lower=-0.52 upper=0.52 effort=1000 velocity=1000 -> lower=-0.495 upper=0.495 effort=0.2 velocity=8.115781022
- joint F3J3: limit lower=-0.52 upper=1.83 effort=1000 velocity=1000 -> lower=-0.4932 upper=1.6272 effort=0.3 velocity=12.86307659
- joint F3J4: limit lower=-0.52 upper=1.83 effort=1000 velocity=1000 -> lower=-0.4932 upper=1.6272 effort=0.3 velocity=13.57866158
- joint F4J1: axis 0 0 1 -> 0 0 -1; limit lower=-0.52 upper=1.83 effort=1000 velocity=1000 -> lower=-1.63595 upper=0.32695 effort=1.0 velocity=8.203047484
- joint F4J2: axis 0 -1 0 -> 0 1 0; limit lower=-0.52 upper=0.52 effort=1000 velocity=1000 -> lower=-0.495 upper=0.495 effort=0.2 velocity=8.115781022
- joint F4J3: limit lower=-0.52 upper=1.83 effort=1000 velocity=1000 -> lower=-0.4932 upper=1.6272 effort=0.3 velocity=12.86307659
- joint F4J4: limit lower=-0.52 upper=1.83 effort=1000 velocity=1000 -> lower=-0.4932 upper=1.6272 effort=0.3 velocity=13.57866158
- joint F5J1: axis 0 0 1 -> 0 0 -1; limit lower=-0.52 upper=1.83 effort=1000 velocity=1000 -> lower=-1.63595 upper=0.32695 effort=1.0 velocity=8.203047484
- joint F5J2: axis 0 -1 0 -> 0 1 0; limit lower=-0.52 upper=0.52 effort=1000 velocity=1000 -> lower=-0.495 upper=0.495 effort=0.2 velocity=8.115781022
- joint F5J3: limit lower=-0.52 upper=1.83 effort=1000 velocity=1000 -> lower=-0.4932 upper=1.6272 effort=0.3 velocity=12.86307659
- joint F5J4: limit lower=-0.52 upper=1.83 effort=1000 velocity=1000 -> lower=-0.4932 upper=1.6272 effort=0.3 velocity=13.57866158
- joint fingertip_ring_fixed: limit lower=0 upper=0 effort=0 velocity=0 -> (none)

File: right_hands/urdf/d5_right_hands_tips.urdf (robot description, URDF)
Before this commit: robot d5_right_hands_tips, 26 links, 25 joints
Joints:
- joint F1J1: axis 0 0 -1 -> 0 0 1; limit lower=-1.83 upper=1 effort=1000 velocity=1000 -> lower=-0.0448 upper=1.6508 effort=0.6 velocity=8.58701992
- joint F1J2: axis 0 1 0 -> 0 -1 0; limit lower=-0.47 upper=1.73 effort=1000 velocity=1000 -> lower=-0.1659 upper=0.9339 effort=0.6 velocity=11.10029404
- joint F1J3: axis 0 0 -1 -> 0 0 1; limit lower=-1.83 upper=0.52 effort=1000 velocity=1000 -> lower=-0.4932 upper=1.6272 effort=0.3 velocity=12.86307659
- joint F1J4: axis 0 0 -1 -> 0 0 1; limit lower=-1.74 upper=0.61 effort=1000 velocity=1000 -> lower=-0.4932 upper=1.6272 effort=0.3 velocity=13.57866158
- joint F2J1: axis 0 0 1 -> 0 0 -1; limit lower=-0.52 upper=1.83 effort=1000 velocity=1000 -> lower=-1.63595 upper=0.32695 effort=1.0 velocity=8.203047484
- joint F2J2: axis 0 -1 0 -> 0 1 0; limit lower=-0.52 upper=0.52 effort=1000 velocity=1000 -> lower=-0.495 upper=0.495 effort=0.2 velocity=8.115781022
- joint F2J3: limit lower=-0.52 upper=1.83 effort=1000 velocity=1000 -> lower=-0.4932 upper=1.6272 effort=0.3 velocity=12.86307659
- joint F2J4: limit lower=-0.52 upper=1.74 effort=1000 velocity=1000 -> lower=-0.4932 upper=1.6272 effort=0.3 velocity=13.57866158
- joint F3J1: axis 0 0 1 -> 0 0 -1; limit lower=-0.52 upper=1.83 effort=1000 velocity=1000 -> lower=-1.63595 upper=0.32695 effort=1.0 velocity=8.203047484
- joint F3J2: axis 0 -1 0 -> 0 1 0; limit lower=-0.52 upper=0.52 effort=1000 velocity=1000 -> lower=-0.495 upper=0.495 effort=0.2 velocity=8.115781022
- joint F3J3: limit lower=-0.52 upper=1.83 effort=1000 velocity=1000 -> lower=-0.4932 upper=1.6272 effort=0.3 velocity=12.86307659
- joint F3J4: limit lower=-0.52 upper=1.83 effort=1000 velocity=1000 -> lower=-0.4932 upper=1.6272 effort=0.3 velocity=13.57866158
- joint F4J1: axis 0 0 1 -> 0 0 -1; limit lower=-0.52 upper=1.83 effort=1000 velocity=1000 -> lower=-1.63595 upper=0.32695 effort=1.0 velocity=8.203047484
- joint F4J2: axis 0 -1 0 -> 0 1 0; limit lower=-0.52 upper=0.52 effort=1000 velocity=1000 -> lower=-0.495 upper=0.495 effort=0.2 velocity=8.115781022
- joint F4J3: limit lower=-0.52 upper=1.83 effort=1000 velocity=1000 -> lower=-0.4932 upper=1.6272 effort=0.3 velocity=12.86307659
- joint F4J4: limit lower=-0.52 upper=1.83 effort=1000 velocity=1000 -> lower=-0.4932 upper=1.6272 effort=0.3 velocity=13.57866158
- joint F5J1: axis 0 0 1 -> 0 0 -1; limit lower=-0.52 upper=1.83 effort=1000 velocity=1000 -> lower=-1.63595 upper=0.32695 effort=1.0 velocity=8.203047484
- joint F5J2: axis 0 -1 0 -> 0 1 0; limit lower=-0.52 upper=0.52 effort=1000 velocity=1000 -> lower=-0.495 upper=0.495 effort=0.2 velocity=8.115781022
- joint F5J3: limit lower=-0.52 upper=1.83 effort=1000 velocity=1000 -> lower=-0.4932 upper=1.6272 effort=0.3 velocity=12.86307659
- joint F5J4: limit lower=-0.52 upper=1.83 effort=1000 velocity=1000 -> lower=-0.4932 upper=1.6272 effort=0.3 velocity=13.57866158
- joint fingertip_ring_fixed: limit lower=0 upper=0 effort=0 velocity=0 -> (none)

Commit message: feat(urdf): Unified the positive direction of the joints
- Adapt to the latest SDK

File: left_hands/d5_left_hands_tips.urdf (robot description, URDF)
Before this commit: robot d5_left_hands_tips, 26 links, 25 joints
Joints:
- joint F2J1: axis 0 0 -1 -> 0 0 1; limit lower=-1.63595 upper=0.32695 effort=1.0 velocity=8.203047484 -> lower=-0.32695 upper=1.63595 effort=1.0 velocity=8.203047484
- joint F3J1: axis 0 0 -1 -> 0 0 1; limit lower=-1.63595 upper=0.32695 effort=1.0 velocity=8.203047484 -> lower=-0.32695 upper=1.63595 effort=1.0 velocity=8.203047484
- joint F4J1: axis 0 0 -1 -> 0 0 1; limit lower=-1.63595 upper=0.32695 effort=1.0 velocity=8.203047484 -> lower=-0.32695 upper=1.63595 effort=1.0 velocity=8.203047484
- joint F5J1: axis 0 0 -1 -> 0 0 1; limit lower=-1.63595 upper=0.32695 effort=1.0 velocity=8.203047484 -> lower=-0.32695 upper=1.63595 effort=1.0 velocity=8.203047484

File: left_hands/urdf/d5_left_hands_tips.urdf (robot description, URDF)
Before this commit: robot d5_left_hands_tips, 26 links, 25 joints
Joints:
- joint F2J1: axis 0 0 -1 -> 0 0 1; limit lower=-1.63595 upper=0.32695 effort=1.0 velocity=8.203047484 -> lower=-0.32695 upper=1.63595 effort=1.0 velocity=8.203047484
- joint F3J1: axis 0 0 -1 -> 0 0 1; limit lower=-1.63595 upper=0.32695 effort=1.0 velocity=8.203047484 -> lower=-0.32695 upper=1.63595 effort=1.0 velocity=8.203047484
- joint F4J1: axis 0 0 -1 -> 0 0 1; limit lower=-1.63595 upper=0.32695 effort=1.0 velocity=8.203047484 -> lower=-0.32695 upper=1.63595 effort=1.0 velocity=8.203047484
- joint F5J1: axis 0 0 -1 -> 0 0 1; limit lower=-1.63595 upper=0.32695 effort=1.0 velocity=8.203047484 -> lower=-0.32695 upper=1.63595 effort=1.0 velocity=8.203047484

File: right_hands/d5_right_hands_tips.urdf (robot description, URDF)
Before this commit: robot d5_right_hands_tips, 26 links, 25 joints
Joints:
- joint F2J1: axis 0 0 -1 -> 0 0 1; limit lower=-1.63595 upper=0.32695 effort=1.0 velocity=8.203047484 -> lower=-0.32695 upper=1.63595 effort=1.0 velocity=8.203047484
- joint F3J1: axis 0 0 -1 -> 0 0 1; limit lower=-1.63595 upper=0.32695 effort=1.0 velocity=8.203047484 -> lower=-0.32695 upper=1.63595 effort=1.0 velocity=8.203047484
- joint F4J1: axis 0 0 -1 -> 0 0 1; limit lower=-1.63595 upper=0.32695 effort=1.0 velocity=8.203047484 -> lower=-0.32695 upper=1.63595 effort=1.0 velocity=8.203047484
- joint F5J1: axis 0 0 -1 -> 0 0 1; limit lower=-1.63595 upper=0.32695 effort=1.0 velocity=8.203047484 -> lower=-0.32695 upper=1.63595 effort=1.0 velocity=8.203047484

File: right_hands/urdf/d5_right_hands_tips.urdf (robot description, URDF)
Before this commit: robot d5_right_hands_tips, 26 links, 25 joints
Joints:
- joint F2J1: axis 0 0 -1 -> 0 0 1; limit lower=-1.63595 upper=0.32695 effort=1.0 velocity=8.203047484 -> lower=-0.32695 upper=1.63595 effort=1.0 velocity=8.203047484
- joint F3J1: axis 0 0 -1 -> 0 0 1; limit lower=-1.63595 upper=0.32695 effort=1.0 velocity=8.203047484 -> lower=-0.32695 upper=1.63595 effort=1.0 velocity=8.203047484
- joint F4J1: axis 0 0 -1 -> 0 0 1; limit lower=-1.63595 upper=0.32695 effort=1.0 velocity=8.203047484 -> lower=-0.32695 upper=1.63595 effort=1.0 velocity=8.203047484
- joint F5J1: axis 0 0 -1 -> 0 0 1; limit lower=-1.63595 upper=0.32695 effort=1.0 velocity=8.203047484 -> lower=-0.32695 upper=1.63595 effort=1.0 velocity=8.203047484
