Commit message: fix: Incorrect mass & inertial of `MCP_joint_pinky`

File: right_hands/d5_right_hands_tips.urdf (robot description, URDF)
Before this commit: robot d5_right_hands_tips, 26 links, 25 joints
Links:
- link MCP_joint_pinky: mass 0 -> 0.000379025355832582

File: right_hands/urdf/d5_right_hands_tips.urdf (robot description, URDF)
Before this commit: robot d5_right_hands_tips, 26 links, 25 joints
Links:
- link MCP_joint_pinky: mass 0 -> 0.000379025355832582
