Commit message: Tempory limit update

File: urdf/left.urdf (robot description, URDF)
Before this commit: robot wujihand-left-v1.0.0, 26 links, 25 joints
Joints:
- joint finger1_joint3: limit lower=-0.4932 upper=1.6272 effort=0.3 velocity=12.86307659 -> lower=0.1 upper=1.6272 effort=0.3 velocity=12.86307659
- joint finger1_joint4: limit lower=-0.4932 upper=1.6272 effort=0.3 velocity=13.57866158 -> lower=0.1 upper=1.6272 effort=0.3 velocity=13.57866158

File: urdf/right.urdf (robot description, URDF)
Before this commit: robot wujihand-right-v1.0.0, 26 links, 25 joints
Joints:
- joint finger1_joint3: limit lower=-0.4932 upper=1.6272 effort=0.3 velocity=12.86307659 -> lower=0.1 upper=1.6272 effort=0.3 velocity=12.86307659
- joint finger1_joint4: limit lower=-0.4932 upper=1.6272 effort=0.3 velocity=13.57866158 -> lower=0.1 upper=1.6272 effort=0.3 velocity=13.57866158

Commit message: refactor: standardize joint and link naming conventions
- Rename fingers from finger1-5 to anatomical names (thumb, index, middle, ring, pinky)
- Standardize joint naming with descriptive axis indicators:
  - {finger}_mcp_pitch_joint (Y-axis flexion/extension)
  - {finger}_mcp_roll_joint (X-axis abduction/adduction)
  - {finger}_pip_joint (proximal interphalangeal)
  - {finger}_dip_joint (distal interphalangeal)
- Add _link suffix to all link names for consistency
- Update all link names to anatomical segments:
  - {finger}_metacarpal_link
  - {finger}_proximal_link
  - {finger}_middle_link
  - {finger}_distal_link
  - {finger}_tip_link
- Rename all 50 mesh files to match new link naming scheme
- Update launch files to use underscores instead of dots

File: urdf/left.urdf (robot description, URDF)
Before this commit: robot wujihand-left-v1.0.0, 26 links, 25 joints
Links:
- removed link finger1_link1
- removed link finger1_link2
- removed link finger1_link3
- removed link finger1_link4
- removed link finger1_tip_link
- removed link finger2_link1
- removed link finger2_link2
- removed link finger2_link3
- removed link finger2_link4
- removed link finger2_tip_link
- removed link finger3_link1
- removed link finger3_link2
- removed link finger3_link3
- removed link finger3_link4
- removed link finger3_tip_link
- removed link finger4_link1
- removed link finger4_link2
- removed link finger4_link3
- removed link finger4_link4
- removed link finger4_tip_link
- removed link finger5_link1
- removed link finger5_link2
- removed link finger5_link3
- removed link finger5_link4
- removed link finger5_tip_link
- added link index_distal_link, mass 0.014; collision mesh filename=package://wujihand-urdf/meshes/left/index_distal_link.STL; visual mesh filename=package://wujihand-urdf/meshes/left/index_distal_link.STL
- added link index_metacarpal_link, mass 0.0032; collision mesh filename=package://wujihand-urdf/meshes/left/index_metacarpal_link.S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; visual mesh filename=package://wujihand-urdf/meshes/left/index_metacarpal_link.S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
- added link index_middle_link, mass 0.0165; collision mesh filename=package://wujihand-urdf/meshes/left/index_middle_link.STL; visual mesh filename=package://wujihand-urdf/meshes/left/index_middle_link.STL
- added link index_proximal_link, mass 0.033; collision mesh filename=package://wujihand-urdf/meshes/left/index_proximal_link.STL; visual mesh filename=package://wujihand-urdf/meshes/left/index_proximal_link.STL
- added link index_tip_link, mass 0.004; collision mesh filename=package://wujihand-urdf/meshes/left/index_tip_link.STL; visual mesh filename=package://wujihand-urdf/meshes/left/index_tip_link.STL
- added link middle_distal_link, mass 0.014; collision mesh filename=package://wujihand-urdf/meshes/left/middle_distal_link.STL; visual mesh filename=package://wujihand-urdf/meshes/left/middle_distal_link.STL
- added link middle_metacarpal_link, mass 0.0032; collision mesh filename=package://wujihand-urdf/meshes/left/middle_metacarpal_link.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; visual mesh filename=package://wujihand-urdf/meshes/left/middle_metacarpal_link.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
- added link middle_middle_link, mass 0.0165; collision mesh filename=package://wujihand-urdf/meshes/left/middle_middle_link.STL; visual mesh filename=package://wujihand-urdf/meshes/left/middle_middle_link.STL
- added link middle_proximal_link, mass 0.033; collision mesh filename=package://wujihand-urdf/meshes/left/middle_proximal_link.STL; visual mesh filename=package://wujihand-urdf/meshes/left/middle_proximal_link.STL
- added link middle_tip_link, mass 0.004; collision mesh filename=package://wujihand-urdf/meshes/left/middle_tip_link.STL; visual mesh filename=package://wujihand-urdf/meshes/left/middle_tip_link.STL
- added link pinky_distal_link, mass 0.014; collision mesh filename=package://wujihand-urdf/meshes/left/pinky_distal_link.STL; visual mesh filename=package://wujihand-urdf/meshes/left/pinky_distal_link.STL
- added link pinky_metacarpal_link, mass 0.0032; collision mesh filename=package://wujihand-urdf/meshes/left/pinky_metacarpal_link.S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; visual mesh filename=package://wujihand-urdf/meshes/left/pinky_metacarpal_link.S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
- added link pinky_middle_link, mass 0.0165; collision mesh filename=package://wujihand-urdf/meshes/left/pinky_middle_link.STL; visual mesh filename=package://wujihand-urdf/meshes/left/pinky_middle_link.STL
- added link pinky_proximal_link, mass 0.033; collision mesh filename=package://wujihand-urdf/meshes/left/pinky_proximal_link.STL; visual mesh filename=package://wujihand-urdf/meshes/left/pinky_proximal_link.STL
- added link pinky_tip_link, mass 0.004; collision mesh filename=package://wujihand-urdf/meshes/left/pinky_tip_link.STL; visual mesh filename=package://wujihand-urdf/meshes/left/pinky_tip_link.STL
- added link ring_distal_link, mass 0.014; collision mesh filename=package://wujihand-urdf/meshes/left/ring_distal_link.STL; visual mesh filename=package://wujihand-urdf/meshes/left/ring_distal_link.STL
- added link ring_metacarpal_link, mass 0.0032; collision mesh filename=package://wujihand-urdf/meshes/left/ring_metacarpal_link.STL; visual mesh filename=package://wujihand-urdf/meshes/left/ring_metacarpal_link.STL
- added link ring_middle_link, mass 0.0165; collision mesh filename=package://wujihand-urdf/meshes/left/ring_middle_link.STL; visual mesh filename=package://wujihand-urdf/meshes/left/ring_middle_link.STL
- added link ring_proximal_link, mass 0.033; collision mesh filename=package://wujihand-urdf/meshes/left/ring_proximal_link.STL; visual mesh filename=package://wujihand-urdf/meshes/left/ring_proximal_link.STL
- added link ring_tip_link, mass 0.004; collision mesh filename=package://wujihand-urdf/meshes/left/ring_tip_link.STL; visual mesh filename=package://wujihand-urdf/meshes/left/ring_tip_link.STL
- added link thumb_distal_link, mass 0.0165; collision mesh filename=package://wujihand-urdf/meshes/left/thumb_distal_link.STL; visual mesh filename=package://wujihand-urdf/meshes/left/thumb_distal_link.STL
- added link thumb_metacarpal_link, mass 0.0075; collision mesh filename=package://wujihand-urdf/meshes/left/thumb_metacarpal_link.S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; visual mesh filename=package://wujihand-urdf/meshes/left/thumb_metacarpal_link.S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
- added link thumb_middle_link, mass 0.0165; collision mesh filename=package://wujihand-urdf/meshes/left/thumb_middle_link.STL; visual mesh filename=package://wujihand-urdf/meshes/left/thumb_middle_link.STL
- added link thumb_proximal_link, mass 0.0248; collision mesh filename=package://wujihand-urdf/meshes/left/thumb_proximal_link.STL; visual mesh filename=package://wujihand-urdf/meshes/left/thumb_proximal_link.STL
- added link thumb_tip_link, mass 0.004; collision mesh filename=package://wujihand-urdf/meshes/left/thumb_tip_link.STL; visual mesh filename=package://wujihand-urdf/meshes/left/thumb_tip_link.STL
Joints:
- removed joint finger1_joint1
- removed joint finger1_joint2
- removed joint finger1_joint3
- removed joint finger1_joint4
- removed joint finger1_tip_fixed
- removed joint finger2_joint1
- removed joint finger2_joint2
- removed joint finger2_joint3
- removed joint finger2_joint4
- removed joint finger2_tip_fixed
- removed joint finger3_joint1
- removed joint finger3_joint2
- removed joint finger3_joint3
- removed joint finger3_joint4
- removed joint finger3_tip_fixed
- removed joint finger4_joint1
- removed joint finger4_joint2
- removed joint finger4_joint3
- removed joint finger4_joint4
- removed joint finger4_tip_fixed
- removed joint finger5_joint1
- removed joint finger5_joint2
- removed joint finger5_joint3
- removed joint finger5_joint4
- removed joint finger5_tip_fixed
- added joint index_dip_joint: type revolute, parent index_middle_link, child index_distal_link, origin xyz=0 0 0.029 rpy=0 0 0, axis -0 1 -0, limit lower=-0.4932 upper=1.6272 effort=0.3 velocity=13.57866158
- added joint index_mcp_pitch_joint: type revolute, parent palm_link, child index_metacarpal_link, origin xyz=-0.0058701 -0.029434 0.091917 rpy=0.11071 -0.071133 0.21823, axis 0 1 0, limit lower=-0.32695 upper=1.63595 effort=1 velocity=8.203047484
- added joint index_mcp_roll_joint: type revolute, parent index_metacarpal_link, child index_proximal_link, origin xyz=0.0022 0 0.004 rpy=-0.00043322 1.0969E-05 0, axis -1 -0 -0, limit lower=-0.495 upper=0.495 effort=0.2 velocity=8.115781022
- added joint index_pip_joint: type revolute, parent index_proximal_link, child index_middle_link, origin xyz=-0.0046 0 0.036618 rpy=0 0 -0.00026861, axis -0 1 -0, limit lower=-0.4932 upper=1.6272 effort=0.3 velocity=12.86307659
- added joint index_tip_fixed: type fixed, parent index_distal_link, child index_tip_link, origin xyz=-0.0010404 0 0.0267 rpy=0 0 0, axis 0 0 0
- added joint middle_dip_joint: type revolute, parent middle_middle_link, child middle_distal_link, origin xyz=0 0 0.029 rpy=0 0 0, axis -0 1 -0, limit lower=-0.4932 upper=1.6272 effort=0.3 velocity=13.57866158
- added joint middle_mcp_pitch_joint: type revolute, parent palm_link, child middle_metacarpal_link, origin xyz=-0.01046 -0.0074615 0.089544 rpy=5.0886E-05 -0.087266 -0.00058387, axis -0 1 -0, limit lower=-0.32695 upper=1.63595 effort=1 velocity=8.203047484
- added joint middle_mcp_roll_joint: type revolute, parent middle_metacarpal_link, child middle_proximal_link, origin xyz=0.0022 0 0.004 rpy=-0.00043323 0 0, axis -1 0 0, limit lower=-0.495 upper=0.495 effort=0.2 velocity=8.115781022
- added joint middle_pip_joint: type revolute, parent middle_proximal_link, child middle_middle_link, origin xyz=-0.0046 0 0.036618 rpy=0 0 -0.00026862, axis -0 1 -0, limit lower=-0.4932 upper=1.6272 effort=0.3 velocity=12.86307659
- added joint middle_tip_fixed: type fixed, parent middle_distal_link, child middle_tip_link, origin xyz=-0.0010404 0 0.0267 rpy=0 0 0, axis 0 0 0
- added joint pinky_dip_joint: type revolute, parent pinky_middle_link, child pinky_distal_link, origin xyz=0 0 0.029 rpy=0 0 0, axis -0 1 -0, limit lower=-0.4932 upper=1.6272 effort=0.3 velocity=13.57866158
- added joint pinky_mcp_pitch_joint: type revolute, parent palm_link, child pinky_metacarpal_link, origin xyz=-0.0022687 0.034001 0.074281 rpy=-0.1925 -0.09326 -0.15753, axis 0 1 0, limit lower=-0.32695 upper=1.63595 effort=1 velocity=8.203047484
- added joint pinky_mcp_roll_joint: type revolute, parent pinky_metacarpal_link, child pinky_proximal_link, origin xyz=0.002203 0 0.0039983 rpy=-0.00043323 0.00075655 0, axis -1 0 0, limit lower=-0.495 upper=0.495 effort=0.2 velocity=8.115781022
- added joint pinky_pip_joint: type revolute, parent pinky_proximal_link, child pinky_middle_link, origin xyz=-0.0046 0 0.036618 rpy=0 0 -0.00026862, axis -0 1 -0, limit lower=-0.4932 upper=1.6272 effort=0.3 velocity=12.86307659
- added joint pinky_tip_fixed: type fixed, parent pinky_distal_link, child pinky_tip_link, origin xyz=-0.0011127 0 0.026697 rpy=0 0 0, axis 0 0 0, limit effort=100 velocity=10
- added joint ring_dip_joint: type revolute, parent ring_middle_link, child ring_distal_link, origin xyz=0 0 0.029 rpy=0 0 0, axis -0 1 -0, limit lower=-0.4932 upper=1.6272 effort=0.3 velocity=13.57866158
- added joint ring_mcp_pitch_joint: type revolute, parent palm_link, child ring_metacarpal_link, origin xyz=-0.0076649 0.013712 0.084429 rpy=-0.090379 -0.084038 -0.047072, axis -0 1 -0, limit lower=-0.32695 upper=1.63595 effort=1 velocity=8.203047484
- added joint ring_mcp_roll_joint: type revolute, parent ring_metacarpal_link, child ring_proximal_link, origin xyz=0.0022024 0 0.0039987 rpy=-0.00043323 0.00060486 0, axis -1 0 0, limit lower=-0.495 upper=0.495 effort=0.2 velocity=8.115781022
- added joint ring_pip_joint: type revolute, parent ring_proximal_link, child ring_middle_link, origin xyz=-0.0046 0 0.036618 rpy=0 0 -0.00026862, axis -0 1 -0, limit lower=-0.4932 upper=1.6272 effort=0.3 velocity=12.86307659
- added joint ring_tip_fixed: type fixed, parent ring_distal_link, child ring_tip_link, origin xyz=-0.0010993 0 0.026698 rpy=0 0 0, axis 0 0 0
- added joint thumb_dip_joint: type revolute, parent thumb_middle_link, child thumb_distal_link, origin xyz=0 4.0225E-05 0.028987 rpy=0 0 0, axis 0 1 0, limit lower=-0.4932 upper=1.6272 effort=0.3 velocity=13.57866158
- added joint thumb_mcp_pitch_joint: type revolute, parent palm_link, child thumb_metacarpal_link, origin xyz=0.0085244 -0.020575 0.028712 rpy=1.328 -0.37161 0.7307, axis -0 1 -0, limit lower=-0.0448 upper=1.6508 effort=0.6 velocity=8.58701992
- added joint thumb_mcp_roll_joint: type revolute, parent thumb_metacarpal_link, child thumb_proximal_link, origin xyz=-0.0047549 0.0060191 0.014132 rpy=-0.27968 -0.55633 -0.081982, axis -1 0 0, limit lower=-0.1659 upper=0.9339 effort=0.6 velocity=11.10029404
- added joint thumb_pip_joint: type revolute, parent thumb_proximal_link, child thumb_middle_link, origin xyz=0.0009915 -0.00026671 0.033166 rpy=-0.049049 0.017311 0.33774, axis 0 1 0, limit lower=-0.4932 upper=1.6272 effort=0.3 velocity=12.86307659
- added joint thumb_tip_fixed: type fixed, parent thumb_distal_link, child thumb_tip_link, origin xyz=-0.001058 -0.00044022 0.029313 rpy=0 0 0, axis 0 0 0, limit lower=-0.5236 upper=0.5236 effort=100 velocity=10
