Commit message: refactor: standardize joint and link naming conventions
- Rename fingers from finger1-5 to anatomical names (thumb, index, middle, ring, pinky)
- Standardize joint naming with descriptive axis indicators:
  - {finger}_mcp_pitch_joint (Y-axis flexion/extension)
  - {finger}_mcp_roll_joint (X-axis abduction/adduction)
  - {finger}_pip_joint (proximal interphalangeal)
  - {finger}_dip_joint (distal interphalangeal)
- Add _link suffix to all link names for consistency
- Update all link names to anatomical segments:
  - {finger}_metacarpal_link
  - {finger}_proximal_link
  - {finger}_middle_link
  - {finger}_distal_link
  - {finger}_tip_link
- Rename all 50 mesh files to match new link naming scheme
- Update launch files to use underscores instead of dots

File: urdf/right.urdf (robot description, URDF)
Before this commit: robot wujihand-right-v1.0.0, 26 links, 25 joints
Links:
- removed link finger1_link1
- removed link finger1_link2
- removed link finger1_link3
- removed link finger1_link4
- removed link finger1_tip_link
- removed link finger2_link1
- removed link finger2_link2
- removed link finger2_link3
- removed link finger2_link4
- removed link finger2_tip_link
- removed link finger3_link1
- removed link finger3_link2
- removed link finger3_link3
- removed link finger3_link4
- removed link finger3_tip_link
- removed link finger4_link1
- removed link finger4_link2
- removed link finger4_link3
- removed link finger4_link4
- removed link finger4_tip_link
- removed link finger5_link1
- removed link finger5_link2
- removed link finger5_link3
- removed link finger5_link4
- removed link finger5_tip_link
- added link index_distal_link, mass 0.014; collision mesh filename=package://wujihand-urdf/meshes/right/index_distal_link.STL; visual mesh filename=package://wujihand-urdf/meshes/right/index_distal_link.STL
- added link index_metacarpal_link, mass 0.0032; collision mesh filename=package://wujihand-urdf/meshes/right/index_metacarpal_link.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; visual mesh filename=package://wujihand-urdf/meshes/right/index_metacarpal_link.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
- added link index_middle_link, mass 0.0165; collision mesh filename=package://wujihand-urdf/meshes/right/index_middle_link.STL; visual mesh filename=package://wujihand-urdf/meshes/right/index_middle_link.STL
- added link index_proximal_link, mass 0.033; collision mesh filename=package://wujihand-urdf/meshes/right/index_proximal_link.STL; visual mesh filename=package://wujihand-urdf/meshes/right/index_proximal_link.STL
- added link index_tip_link, mass 0.004; collision mesh filename=package://wujihand-urdf/meshes/right/index_tip_link.STL; visual mesh filename=package://wujihand-urdf/meshes/right/index_tip_link.STL
- added link middle_distal_link, mass 0.014; collision mesh filename=package://wujihand-urdf/meshes/right/middle_distal_link.STL; visual mesh filename=package://wujihand-urdf/meshes/right/middle_distal_link.STL
- added link middle_metacarpal_link, mass 0.0032; collision mesh filename=package://wujihand-urdf/meshes/right/middle_metacarpal_link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; visual mesh filename=package://wujihand-urdf/meshes/right/middle_metacarpal_link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
- added link middle_middle_link, mass 0.0165; collision mesh filename=package://wujihand-urdf/meshes/right/middle_middle_link.STL; visual mesh filename=package://wujihand-urdf/meshes/right/middle_middle_link.STL
- added link middle_proximal_link, mass 0.033; collision mesh filename=package://wujihand-urdf/meshes/right/middle_proximal_link.S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; visual mesh filename=package://wujihand-urdf/meshes/right/middle_proximal_link.S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
- added link middle_tip_link, mass 0.004; collision mesh filename=package://wujihand-urdf/meshes/right/middle_tip_link.STL; visual mesh filename=package://wujihand-urdf/meshes/right/middle_tip_link.STL
- added link pinky_distal_link, mass 0.014; collision mesh filename=package://wujihand-urdf/meshes/right/pinky_distal_link.STL; visual mesh filename=package://wujihand-urdf/meshes/right/pinky_distal_link.STL
- added link pinky_metacarpal_link, mass 0.0032; collision mesh filename=package://wujihand-urdf/meshes/right/pinky_metacarpal_link.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; visual mesh filename=package://wujihand-urdf/meshes/right/pinky_metacarpal_link.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
- added link pinky_middle_link, mass 0.0165; collision mesh filename=package://wujihand-urdf/meshes/right/pinky_middle_link.STL; visual mesh filename=package://wujihand-urdf/meshes/right/pinky_middle_link.STL
- added link pinky_proximal_link, mass 0.033; collision mesh filename=package://wujihand-urdf/meshes/right/pinky_proximal_link.STL; visual mesh filename=package://wujihand-urdf/meshes/right/pinky_proximal_link.STL
- added link pinky_tip_link, mass 0.004; collision mesh filename=package://wujihand-urdf/meshes/right/pinky_tip_link.STL; visual mesh filename=package://wujihand-urdf/meshes/right/pinky_tip_link.STL
- added link ring_distal_link, mass 0.014; collision mesh filename=package://wujihand-urdf/meshes/right/ring_distal_link.STL; visual mesh filename=package://wujihand-urdf/meshes/right/ring_distal_link.STL
- added link ring_metacarpal_link, mass 0.0032; collision mesh filename=package://wujihand-urdf/meshes/right/ring_metacarpal_link.S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; visual mesh filename=package://wujihand-urdf/meshes/right/ring_metacarpal_link.S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
- added link ring_middle_link, mass 0.0165; collision mesh filename=package://wujihand-urdf/meshes/right/ring_middle_link.STL; visual mesh filename=package://wujihand-urdf/meshes/right/ring_middle_link.STL
- added link ring_proximal_link, mass 0.033; collision mesh filename=package://wujihand-urdf/meshes/right/ring_proximal_link.STL; visual mesh filename=package://wujihand-urdf/meshes/right/ring_proximal_link.STL
- added link ring_tip_link, mass 0.004; collision mesh filename=package://wujihand-urdf/meshes/right/ring_tip_link.STL; visual mesh filename=package://wujihand-urdf/meshes/right/ring_tip_link.STL
- added link thumb_distal_link, mass 0.0165; collision mesh filename=package://wujihand-urdf/meshes/right/thumb_distal_link.STL; visual mesh filename=package://wujihand-urdf/meshes/right/thumb_distal_link.STL
- added link thumb_metacarpal_link, mass 0.0075; collision mesh filename=package://wujihand-urdf/meshes/right/thumb_metacarpal_link.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; visual mesh filename=package://wujihand-urdf/meshes/right/thumb_metacarpal_link.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
- added link thumb_middle_link, mass 0.0165; collision mesh filename=package://wujihand-urdf/meshes/right/thumb_middle_link.STL; visual mesh filename=package://wujihand-urdf/meshes/right/thumb_middle_link.STL
- added link thumb_proximal_link, mass 0.0248; collision mesh filename=package://wujihand-urdf/meshes/right/thumb_proximal_link.STL; visual mesh filename=package://wujihand-urdf/meshes/right/thumb_proximal_link.STL
- added link thumb_tip_link, mass 0.004; collision mesh filename=package://wujihand-urdf/meshes/right/thumb_tip_link.STL; visual mesh filename=package://wujihand-urdf/meshes/right/thumb_tip_link.STL
Joints:
- removed joint finger1_joint1
- removed joint finger1_joint2
- removed joint finger1_joint3
- removed joint finger1_joint4
- removed joint finger1_tip_fixed
- removed joint finger2_joint1
- removed joint finger2_joint2
- removed joint finger2_joint3
- removed joint finger2_joint4
- removed joint finger2_tip_fixed
- removed joint finger3_joint1
- removed joint finger3_joint2
- removed joint finger3_joint3
- removed joint finger3_joint4
- removed joint finger3_tip_fixed
- removed joint finger4_joint1
- removed joint finger4_joint2
- removed joint finger4_joint3
- removed joint finger4_joint4
- removed joint finger4_tip_fixed
- removed joint finger5_joint1
- removed joint finger5_joint2
- removed joint finger5_joint3
- removed joint finger5_joint4
- removed joint finger5_tip_fixed
- added joint index_dip_joint: type revolute, parent index_middle_link, child index_distal_link, origin xyz=0 0 0.0290000000150095 rpy=0 0 0, axis -0 1 -0, limit lower=-0.4932 upper=1.6272 effort=0.3 velocity=13.57866158
- added joint index_mcp_pitch_joint: type revolute, parent palm_link, child index_metacarpal_link, origin xyz=-0.00587008921485247 0.0294338632809287 0.0919165306699325 rpy=-0.111142508461784 -0.0711392477320386 -0.218224846477167, axis 0 0.999999906158207 0.000433224625971368, limit lower=-0.32695 upper=1.63595 effort=1 velocity=8.203047484
- added joint index_mcp_roll_joint: type revolute, parent index_metacarpal_link, child index_proximal_link, origin xyz=0.00220000017524629 0 0.00400000534382478 rpy=0.000433224548403847 0 0, axis -0.999999999978991 0 0, limit lower=-0.495 upper=0.495 effort=0.2 velocity=8.115781022
- added joint index_pip_joint: type revolute, parent index_proximal_link, child index_middle_link, origin xyz=-0.00460023735005808 1.55817705260984E-05 0.0366176526568538 rpy=-0.000433222790942502 0 -0.000268612691124751, axis -0 1 -0, limit lower=-0.4932 upper=1.6272 effort=0.3 velocity=12.86307659
- added joint index_tip_fixed: type fixed, parent index_distal_link, child index_tip_link, origin xyz=-0.00104999539509563 0 0.0274000004481596 rpy=0 0 0, axis 0 0 0, limit lower=0 upper=0 effort=100 velocity=10
- added joint middle_dip_joint: type revolute, parent middle_middle_link, child middle_distal_link, origin xyz=0 0 0.0290000000150094 rpy=0 0 0, axis -0 1 -0, limit lower=-0.4932 upper=1.6272 effort=0.3 velocity=13.57866158
- added joint middle_mcp_pitch_joint: type revolute, parent palm_link, child middle_metacarpal_link, origin xyz=-0.0104597238611628 0.00746146014385576 0.0895435117703666 rpy=-0.00048411119168703 -0.087266465303481 0.000583871740106801, axis 0 0.999999906158095 0.000433224884501103, limit lower=-0.32695 upper=1.63595 effort=1 velocity=8.203047484
- added joint middle_mcp_roll_joint: type revolute, parent middle_metacarpal_link, child middle_proximal_link, origin xyz=0.0022000005026625 0 0.00400000522628907 rpy=0.000433224806924388 0 0, axis -1 0 0, limit lower=-0.495 upper=0.495 effort=0.2 velocity=8.115781022
- added joint middle_pip_joint: type revolute, parent middle_proximal_link, child middle_middle_link, origin xyz=-0.00460000064410125 1.55817799863825E-05 0.036617682393194 rpy=-0.000433224785853114 0 -0.000268612686864552, axis -0 1 -0, limit lower=-0.4932 upper=1.6272 effort=0.3 velocity=12.86307659
- added joint middle_tip_fixed: type fixed, parent middle_distal_link, child middle_tip_link, origin xyz=-0.00104042865141054 0 0.0267000008801756 rpy=0 0 0, axis 0 0 0, limit lower=0 upper=0 effort=100 velocity=10
- added joint pinky_dip_joint: type revolute, parent pinky_middle_link, child pinky_distal_link, origin xyz=0 0 0.029 rpy=0 0 0, axis -0 1 -0, limit lower=-0.4932 upper=1.6272 effort=0.3 velocity=13.57866158
- added joint pinky_mcp_pitch_joint: type revolute, parent palm_link, child pinky_metacarpal_link, origin xyz=-0.00226865106062467 -0.0340011106648613 0.0742813381426987 rpy=0.192050433506504 -0.0925172356498861 0.157672818297325, axis 0 0.999999906157892 0.000433225353070638, limit lower=-0.32695 upper=1.63595 effort=1 velocity=8.203047484
- added joint pinky_mcp_roll_joint: type revolute, parent pinky_metacarpal_link, child pinky_proximal_link, origin xyz=0.00220000070730803 0 0.00400000490038611 rpy=0.000433225364229257 0 0, axis -1 0 0, limit lower=-0.495 upper=0.495 effort=0.2 velocity=8.115781022
- added joint pinky_pip_joint: type revolute, parent pinky_proximal_link, child pinky_middle_link, origin xyz=-0.0046 1.5582E-05 0.036618 rpy=-0.00043323 0 -0.00026861, axis -0 1 -0, limit lower=-0.4932 upper=1.6272 effort=0.3 velocity=12.86307659
- added joint pinky_tip_fixed: type fixed, parent pinky_distal_link, child pinky_tip_link, origin xyz=-0.00104042861181322 0 0.0267000011472218 rpy=0 0 0, axis 0 0 0, limit lower=0 upper=0 effort=100 velocity=10
- added joint ring_dip_joint: type revolute, parent ring_middle_link, child ring_distal_link, origin xyz=0 0 0.0290000000150089 rpy=0 0 0, axis -0 1 -0, limit lower=-0.4932 upper=1.6272 effort=0.3 velocity=13.57866158
- added joint ring_mcp_pitch_joint: type revolute, parent palm_link, child ring_metacarpal_link, origin xyz=-0.0076648599285041 -0.0137122383759844 0.084428694586379 rpy=0.0899413960034348 -0.0834355049367681 0.0471266288536016, axis 0 0.999999906157892 0.000433225355001288, limit lower=-0.32695 upper=1.63595 effort=1 velocity=8.203047484
- added joint ring_mcp_roll_joint: type revolute, parent ring_metacarpal_link, child ring_proximal_link, origin xyz=0.00220000053755089 0 0.00400000510026774 rpy=0.000433225366118357 0 0, axis -1 0 0, limit lower=-0.495 upper=0.495 effort=0.2 velocity=8.115781022
- added joint ring_pip_joint: type revolute, parent ring_proximal_link, child ring_middle_link, origin xyz=-0.00459999999033558 1.55818004638833E-05 0.0366176824753135 rpy=-0.000433225349833524 0 -0.000268612687102299, axis -0 1 -0, limit lower=-0.4932 upper=1.6272 effort=0.3 velocity=12.86307659
- added joint ring_tip_fixed: type fixed, parent ring_distal_link, child ring_tip_link, origin xyz=-0.00104042861977702 0 0.026700000917914 rpy=0 0 0, axis 0 0 0, limit lower=0 upper=0 effort=100 velocity=10
- added joint thumb_dip_joint: type revolute, parent thumb_middle_link, child thumb_distal_link, origin xyz=0 -5.00007422951686E-05 0.0289999996622586 rpy=0 0 0, axis 0 1 0, limit lower=-0.4932 upper=1.6272 effort=0.3 velocity=13.57866158
- added joint thumb_mcp_pitch_joint: type revolute, parent palm_link, child thumb_metacarpal_link, origin xyz=0.00852444051536966 0.0205754004992104 0.0287119465316217 rpy=-1.32802443797267 -0.371613529401197 -0.730700470955738, axis -0 1 -0, limit lower=-0.0448 upper=1.6508 effort=0.6 velocity=8.58701992
- added joint thumb_mcp_roll_joint: type revolute, parent thumb_metacarpal_link, child thumb_proximal_link, origin xyz=-0.00475489770145063 -0.00601914141399163 0.0141320977109324 rpy=-0.574275025049342 -0.236773483165492 1.80339766411149, axis -0 -1 -0, limit lower=-0.1659 upper=0.9339 effort=0.6 velocity=11.10029404
- added joint thumb_pip_joint: type revolute, parent thumb_proximal_link, child thumb_middle_link, origin xyz=0.00026670985188593 -0.000991501581071832 0.0331656190850421 rpy=0.0490494507279603 0.0173112436656061 -1.90854042682209, axis 0 1 0, limit lower=-0.4932 upper=1.6272 effort=0.3 velocity=12.86307659
- added joint thumb_tip_fixed: type fixed, parent thumb_distal_link, child thumb_tip_link, origin xyz=-0.00104623528319934 0.000443681117589321 0.0293000000558906 rpy=0 0 0, axis 0 0 0, limit lower=0 upper=0 effort=100 velocity=10
